File: hardware-shift/pcb/Flatbox-rev1.1-kicad/Flatbox-rev1_1.kicad_pcb (KiCad board)
At the start: 2 copper layers, 233.7 x 120 mm, 26 parts, among them SW1 SW_Push, SW10 SW_Push, SW11 SW_Push, SW12 SW_Push, SW13 SW_Push, SW14 SW_Push, SW15 SW_Push, SW16 SW_Push, SW17 SW_Push, SW18 SW_Push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

Commit message: new version with modified action keys and parallel R3/shift
Parts:
- added SW1a1: SW_Push, Button_Switch_THT:SW_PUSH_6mm_H5mm, F.Cu at (75.4, 41.5)
- moved SW16 4.27 mm to (213.8, 85.8)
- moved SW12 3.44 mm to (219.5, 55.0)
Connections:
- U1 pad 21: Net-(U1-Pad21) -> unconnected-(U1-Pad21)
- U1 pad 22: Net-(U1-Pad22) -> unconnected-(U1-Pad22)
- U1 pad 24: Net-(U1-Pad24) -> unconnected-(U1-Pad24)
Routing:
- net OPT1: track 147.5 -> 163.6 mm
- net GND: track 762.8 -> 773.6 mm
- net L2: track 170.9 -> 175.1 mm
- net L1: track 139.9 -> 143.4 mm
- net R2: track 140.5 -> 144.0 mm
- net R1: track 111.2 -> 114.5 mm
Other:
- board text added: "Shiftbox"
- board text added: "github.com/xpire/flatbox-shift (cred: jfedor2)"
- board text added: "rev1.1(shift)"
- board text removed: "Flatbox"
- board text removed: "github.com/jfedor2/flatbox"
- board text removed: "rev1.1"

Commit message: parallel action keys
Parts:
- moved SW16 4.27 mm to (213.8, 90.0)
- moved SW12 3.44 mm to (219.5, 58.4)
Routing:
- net L2: track 175.1 -> 170.9 mm
- net L1: track 143.4 -> 139.9 mm
- net R2: track 144.0 -> 140.5 mm
- net R1: track 114.5 -> 111.2 mm
- net GND: track 773.6 -> 775.0 mm

Commit message: 3rd action keys up, top by 3mm, bottom by 4mm
Parts:
- moved SW16 4.27 mm to (213.8, 85.8)
- moved SW12 3.44 mm to (219.5, 55.0)
Routing:
- net L2: track 170.9 -> 175.1 mm
- net L1: track 139.9 -> 143.4 mm
- net R2: track 140.5 -> 144.0 mm
- net R1: track 111.2 -> 114.5 mm
- net GND: track 775.0 -> 773.6 mm

Commit message: smaller tolerance tilted
Parts:
- moved REF** 6.60 mm to (45.0, 42.0)
- moved REF** 6.60 mm to (45.0, 148.0)
- moved SW13 4.01 mm to (244.4, 58.7)
- moved SW17 4.01 mm to (239.0, 90.0)
- moved SW12 2.48 mm to (217.0, 55.0)
- moved SW16 1.76 mm to (212.0, 85.8)
- moved SW11 1.51 mm to (189.0, 58.6)
- moved SW15 1.22 mm to (183.7, 90.0)
Routing:
- net GND: track 773.6 -> 764.9 mm
- net R2: track 144.0 -> 138.0 mm
- net R1: track 114.5 -> 109.4 mm
- net L1: track 143.4 -> 141.7 mm
- net CIRCLE: track 98.7 -> 97.2 mm
Other:
- board size 233.7 x 120 mm -> 227.1 x 120 mm
- board text added: "circle"
- board text added: "cross"
- board text added: "down"
- board text added: "l1"
- board text added: "l2"
- board text added: "l3"
- board text added: "left"
- board text added: "r1"
- board text added: "r2"
- board text added: "r3"
- board text added: "right"
- board text added: "square"
- board text added: "triangle"
- board text added: "up"

Commit message: added key labels
Other:
- board text added: "1"
- board text added: "2"
- board text added: "3"
- board text added: "4"
- board text added: "5"
- board text added: "6"
- board text added: "shift"
- board text removed: "l3"
- board text removed: "r3"
Changed lines of the file:
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@@
     (effects (font (size 1.5 1.5) (thickness 0.3)))
   )
-  (gr_text "l3" (at 53.1876 107.8784) (layer "F.SilkS")
+  (gr_text "shift" (at 53.1876 107.8784) (layer "F.SilkS")
     (effects (font (size 1.5 1.5) (thickness 0.3)))
   )
@@
     (effects (font (size 2 2) (thickness 0.3)))
   )
-  (gr_text "l3" (at 73.1012 37.7284) (layer "F.SilkS")
+  (gr_text "1" (at 73.1012 37.7284) (layer "F.SilkS")
     (effects (font (size 1.5 1.5) (thickness 0.3)))
   )
   (gr_text "cross" (at 158.3376 115.1284) (layer "F.SilkS")
+    (effects (font (size 1.5 1.5) (thickness 0.3)))
+  )
+  (gr_text "4" (at 105.8376 37.7284) (layer "F.SilkS")
+    (effects (font (size 1.5 1.5) (thickness 0.3)))
+  )
+  (gr_text "5" (at 115.8376 37.7284) (layer "F.SilkS")
     (effects (font (size 1.5 1.5) (thickness 0.3)))
   )
@@
     (effects (font (size 1.5 1.5) (thickness 0.3)))
   )
+  (gr_text "6" (at 125.8376 37.7284) (layer "F.SilkS")
+    (effects (font (size 1.5 1.5) (thickness 0.3)))
+  )
   (gr_text "Shiftbox" (at 222.25 135.89) (layer "F.SilkS")
     (effects (font (size 8 8) (thickness 1)))
@@
     (effects (font (size 1.5 1.5) (thickness 0.3)))
   )
-  (gr_text "r3" (at 82.8376 37.7284) (layer "F.SilkS")
+  (gr_text "3" (at 92.8376 37.7284) (layer "F.SilkS")
     (effects (font (size 1.5 1.5) (thickness 0.3)))
   )
+  (gr_text "2" (at 82.8376 37.7284) (layer "F.SilkS")
+    (effects (font (size 1.5 1.5) (thickness 0.3)))
+  )
