File: hardware-shift-rev2/extras/Flatbox-rev1.1-kicad/Flatbox-rev1_1.kicad_sch (KiCad schematic)
At the start: 20 parts

Commit message: finalised MX compatiable hotswap pcb
Parts:
- SW1, SW2, SW3, SW4, SW5, SW6: value (none) -> SW_Push
- SW10, SW11, SW12, SW13, SW14, SW15, SW16, SW17, SW18, SW7, SW8, SW9: value (none) -> SW_Push; footprint Kailh:Kailh_socket_PG1350_optional -> Switch_Keyboard_Hotswap_Kailh:SW_Hotswap_Kailh_MX_plated_1.00u
- SW19: renamed from SW?; footprint Kailh:Kailh_socket_PG1350_optional -> Switch_Keyboard_Hotswap_Kailh:SW_Hotswap_Kailh_MX_plated_1.00u
- U1: value (none) -> ProMicro
